Commit message: correções a fisicas

File: src/description/gazebo_control.xacro (robot description, xacro)
@@ -2,21 +2,81 @@
 <robot xmlns:xacro="http://www.ros.org/wiki/xacro">
     <!-- Gazebo Harmonic (gz sim), o par do ROS 2 Jazzy -->
-    <!-- Esferas sem atrito para deslizarem -->
-    <gazebo reference="caster_a">
-        <mu1>0.0</mu1>
-        <mu2>0.0</mu2>
+    <!-- ===== Parametros do sensor (RPLIDAR A1M8) =====
+         Datasheet: alcance 0.15 m a 12 m (versoes R5/R6; R4 e inferiores 6 m), >= 8000 amostras/s,
+         5.5 Hz tipico (2-10 Hz), resolucao angular <= 1 grau, erro < 1 % da distancia.
+         Valores abaixo = saida tipica do driver rplidar_ros em A1: 360 pontos a 10 Hz. -->
+    <xacro:property name="lidar_samples" value="360"/>
+    <xacro:property name="lidar_rate" value="10"/>
+    <xacro:property name="lidar_min_range" value="0.15"/>
+    <xacro:property name="lidar_max_range" value="12.0"/>
+    <xacro:property name="lidar_noise_std" value="0.005"/>
+    <!-- ===== Atrito =====
+         Os links filhos de juntas fixas seriam fundidos no pai pelo conversor URDF->SDF e o atrito
+         das esferas perdia-se. preserveFixedJoint mantem as esferas como links proprios. -->
+    <gazebo reference="caster_front_joint"><preserveFixedJoint>true</preserveFixedJoint></gazebo>
+    <gazebo reference="caster_rear_joint"><preserveFixedJoint>true</preserveFixedJoint></gazebo>
+    <!-- esferas livres: sem atrito (rolam em qualquer direcao) -->
+    <gazebo reference="caster_front">
+        <mu1>0.0</mu1><mu2>0.0</mu2>
     </gazebo>
-    <gazebo reference="caster_b">
-        <mu1>0.0</mu1>
-        <mu2>0.0</mu2>
+    <gazebo reference="caster_rear">
+        <mu1>0.0</mu1><mu2>0.0</mu2>
     </gazebo>
-    <gazebo reference="left_wheel"><mu1>1.0</mu1><mu2>1.0</mu2></gazebo>
-    <gazebo reference="right_wheel"><mu1>1.0</mu1><mu2>1.0</mu2></gazebo>
+    <!-- pneus (borracha/TPU sobre papel/vinil do tapete): atrito alto, sem escorregar -->
+    <gazebo reference="left_wheel">
+        <mu1>1.0</mu1><mu2>1.0</mu2>
+    </gazebo>
+    <gazebo reference="right_wheel">
+        <mu1>1.0</mu1><mu2>1.0</mu2>
+    </gazebo>
+    <!-- chassis nao deve ter atrito alto se bater numa parede -->
+    <gazebo reference="chassis">
+        <mu1>0.3</mu1><mu2>0.3</mu2>
+    </gazebo>
+    <!-- ===== LIDAR ===== -->
+    <gazebo reference="laser_frame">
+        <sensor name="rplidar" type="gpu_lidar">
+            <pose>0 0 0 0 0 0</pose>
+            <topic>scan</topic>
+            <gz_frame_id>laser_frame</gz_frame_id>
+            <update_rate>${lidar_rate}</update_rate>
+            <always_on>true</always_on>
+            <visualize>true</visualize>
+            <lidar>
+                <scan>
+                    <horizontal>
+                        <samples>${lidar_samples}</samples>
+                        <resolution>1</resolution>
+                        <min_angle>${-pi}</min_angle>
+                        <max_angle>${pi}</max_angle>
+                    </horizontal>
+                    <!-- plano unico (2D) -->
+                    <vertical>
+                        <samples>1</samples>
+                        <resolution>1</resolution>
+                        <min_angle>0</min_angle>
+                        <max_angle>0</max_angle>
+                    </vertical>
+                </scan>
+                <range>
+                    <min>${lidar_min_range}</min>
+                    <max>${lidar_max_range}</max>
+                    <resolution>0.001</resolution>
+                </range>
+                <noise>
+                    <type>gaussian</type>
+                    <mean>0.0</mean>
+                    <stddev>${lidar_noise_std}</stddev>
+                </noise>
+            </lidar>
+        </sensor>
+    </gazebo>
+    <!-- ===== Controlo diferencial + estado das juntas ===== -->
     <gazebo>
         <plugin filename="gz-sim-diff-drive-system" name="gz::sim::systems::DiffDrive">
             <left_joint>left_wheel_joint</left_joint>
             <right_joint>right_wheel_joint</right_joint>
-            <!-- distancia entre os centros das rodas, medida no CAD -->
-            <wheel_separation>0.0907</wheel_separation>
+            <!-- distancia entre os centros dos pneus, medida no CAD (90.8 mm) -->
+            <wheel_separation>${wheel_separation}</wheel_separation>
             <wheel_radius>${wheel_radius}</wheel_radius>
             <frame_id>odom</frame_id>
@@ -25,6 +85,19 @@
             <odom_topic>odom</odom_topic>
             <tf_topic>tf</tf_topic>
+            <odom_publish_frequency>50</odom_publish_frequency>
+            <!-- limites coerentes com o motor (ver motor_max_speed em robot_core.xacro) -->
+            <max_linear_velocity>${0.9*motor_max_speed*wheel_radius}</max_linear_velocity>
+            <min_linear_velocity>${-0.9*motor_max_speed*wheel_radius}</min_linear_velocity>
+            <max_angular_velocity>${0.9*2*motor_max_speed*wheel_radius/wheel_separation}</max_angular_velocity>
+            <min_angular_velocity>${-0.9*2*motor_max_speed*wheel_radius/wheel_separation}</min_angular_velocity>
+            <max_linear_acceleration>2.0</max_linear_acceleration>
+            <min_linear_acceleration>-2.0</min_linear_acceleration>
+            <max_angular_acceleration>12.0</max_angular_acceleration>
+            <min_angular_acceleration>-12.0</min_angular_acceleration>
         </plugin>
+        <!-- topic explicito: por omissao o gz publica em /world/<mundo>/model/<nome>/joint_state
+             e a ponte para /joint_states nunca recebia nada (sem TF das rodas no RViz) -->
         <plugin filename="gz-sim-joint-state-publisher-system" name="gz::sim::systems::JointStatePublisher">
+            <topic>joint_states</topic>
             <joint_name>left_wheel_joint</joint_name>
             <joint_name>right_wheel_joint</joint_name>

File: src/description/robot_core.xacro (robot description, xacro)
@@ -1,4 +1,14 @@
 <?xml version="1.0"?>
 <robot xmlns:xacro="http://www.ros.org/wiki/xacro">
+    <!-- =====================================================================
+         FRAMES (convencao ROS, REP-103)
+           base_link : ponto medio do eixo das rodas, a altura do eixo
+                       (x = frente, y = esquerda, z = cima)
+           chassis   : "plate frame" = frame da placa base no CAD (frente = -Y).
+                       E o frame em que estao todas as poses das meshes.
+         Todas as poses das meshes foram recalculadas relativamente a placa base:
+         o export do Onshape vinha rodado 2.4 graus em Z / 1 grau em Y, o que
+         deixava os eixos das rodas tortos e o robo a andar ligeiramente de lado.
+         ===================================================================== -->
     <!-- ================= MATERIAIS ================= -->
     <material name="white"><color rgba="1 1 1 1"/></material>
@@ -8,16 +18,38 @@
     <material name="grey"><color rgba="0.7 0.7 0.7 1"/></material>
     <material name="light_blue"><color rgba="0.62 0.81 0.93 1"/></material>
-    <!-- ================= PARAMETROS ================= -->
-    <!-- medidos no roda.stl: diametro 56 mm, largura 8 mm -->
-    <xacro:property name="wheel_radius" value="0.028"/>
-    <xacro:property name="wheel_width" value="0.008"/>
-    <xacro:property name="wheel_mass" value="0.03"/>
-    <xacro:property name="chassis_mass" value="0.5"/>
-    <xacro:property name="caster_ball_radius" value="0.006"/>   <!-- bola de 12 mm -->
+    <!-- ================= PARAMETROS GEOMETRICOS (medidos no CAD) ================= -->
     <xacro:property name="meshes" value="package://my_bot/description/meshes"/>
-    <!-- No CAD a frente do robo e -Y. Rodar +90 graus em Z poe a frente em +X (convencao ROS). -->
-    <xacro:property name="chassis_yaw" value="${pi/2}"/>
-    <!-- centro da mesh do LIDAR no frame do chassis, calculado a partir do export (assenta no topo do 'resto') -->
-    <xacro:property name="lidar_xyz" value="0.0001 -0.0084 0.0913"/>
+    <xacro:property name="wheel_radius" value="0.028"/>            <!-- roda.stl: diametro 56 mm -->
+    <xacro:property name="wheel_width" value="0.008"/>             <!-- roda.stl: 8 mm -->
+    <xacro:property name="wheel_y" value="0.0454"/>                <!-- centro de cada roda (CAD: separacao centro-a-centro 90.8 mm) -->
+    <xacro:property name="wheel_separation" value="${2*wheel_y}"/> <!-- 0.0908 m, usado pelo diff_drive -->
+    <xacro:property name="axle_height_in_plate" value="0.007"/>    <!-- eixo das rodas 7 mm acima da origem da placa -->
+    <xacro:property name="caster_ball_radius" value="0.006"/>      <!-- bola de 12 mm -->
+    <!-- esferas: centro a z=-15 mm na placa => fundo a -21 mm == fundo das rodas (7-28 = -21 mm). Os 3 apoios ficam coplanares. -->
+    <xacro:property name="caster_z" value="-0.015"/>
+    <xacro:property name="caster_front_y" value="-0.03813"/>
+    <xacro:property name="caster_rear_y" value="0.03615"/>
+    <!-- ================= PARAMETROS FISICOS (ESTIMATIVAS - pesar o robo e ajustar!) =================
+         Correr  python3 tools/mass_budget.py  para recalcular massa/CM/inercia do chassis
+         depois de mudar a tabela de massas nesse script. -->
+    <xacro:property name="wheel_mass" value="0.012"/>              <!-- roda impressa 7.6 g (PLA macico) + pneu -->
+    <xacro:property name="caster_ball_mass" value="0.0071"/>       <!-- esfera de aco 12 mm: 0.902 cm3 x 7.85 g/cm3 -->
+    <xacro:property name="chassis_mass" value="0.485"/>            <!-- placa 60 g + corpo/bateria/PCBs 200 g + 2 motores + iman + LIDAR 170 g + 2 corpos de caster -->
+    <xacro:property name="chassis_com" value="-0.00006 -0.00094 0.05392"/>
+    <xacro:property name="chassis_ixx" value="1.0369e-03"/>
+    <xacro:property name="chassis_ixy" value="1.6735e-07"/>
+    <xacro:property name="chassis_ixz" value="1.1116e-06"/>
+    <xacro:property name="chassis_iyy" value="8.5370e-04"/>
+    <xacro:property name="chassis_iyz" value="-1.1292e-04"/>
+    <xacro:property name="chassis_izz" value="6.0338e-04"/>
+    <!-- limites do motor (N20 com redutora - ajustar ao motor real) -->
+    <xacro:property name="motor_max_torque" value="0.1"/>          <!-- N.m por roda -->
+    <xacro:property name="motor_max_speed" value="20.0"/>          <!-- rad/s por roda (~190 rpm => 0.56 m/s) -->
+    <!-- ================= LIDAR (RPLIDAR A1) ================= -->
+    <!-- Eixo de rotacao da cabeca medido na mesh: (0, +12.4 mm) no plate frame, i.e. 12.4 mm ATRAS do centro do robo.
+         Plano de varrimento: a meio da cabeca (z = 109 mm na placa). Ajustar se o datasheet indicar outra altura. -->
+    <xacro:property name="lidar_x" value="-0.0124"/>               <!-- em base_link -->
+    <xacro:property name="lidar_y" value="0.0"/>
+    <xacro:property name="lidar_z" value="${0.109 - axle_height_in_plate}"/>
     <!-- ================= MACROS ================= -->
     <xacro:macro name="chassis_visual" params="mesh xyz rpy material:=light_blue">
@@ -28,14 +60,14 @@
         </visual>
     </xacro:macro>
-    <xacro:macro name="wheel" params="name xyz rpy axis">
+    <!-- Roda: origem no centro do pneu, eixo de rotacao = Z do link = +Y do base_link.
+         Velocidade positiva nas duas juntas => robo anda para a frente (+X). -->
+    <xacro:macro name="wheel" params="name y vis_z vis_roll">
         <link name="${name}_wheel">
             <visual>
-                <origin xyz="0 0 0" rpy="-3.14159 0 0"/>
+                <origin xyz="0 0 ${vis_z}" rpy="${vis_roll} 0 0"/>
                 <geometry><mesh filename="${meshes}/roda.stl"/></geometry>
                 <material name="black"/>
             </visual>
             <collision>
-                <!-- cilindro simples (eixo Z = eixo de rotacao); a mesh vai de z=0 a z=-0.008 no frame da roda -->
-                <origin xyz="0 0 ${-wheel_width/2}" rpy="0 0 0"/>
                 <geometry><cylinder radius="${wheel_radius}" length="${wheel_width}"/></geometry>
             </collision>
@@ -48,14 +80,16 @@
         </link>
         <joint name="${name}_wheel_joint" type="continuous">
-            <parent link="chassis"/>
+            <parent link="base_link"/>
             <child link="${name}_wheel"/>
-            <origin xyz="${xyz}" rpy="${rpy}"/>
-            <axis xyz="${axis}"/>
+            <origin xyz="0 ${y} 0" rpy="${-pi/2} 0 0"/>
+            <axis xyz="0 0 1"/>
+            <limit effort="${motor_max_torque}" velocity="${motor_max_speed}"/>
+            <dynamics damping="0.0005" friction="0.0"/>
         </joint>
     </xacro:macro>
-    <xacro:macro name="caster_ball" params="name xyz rpy">
+    <!-- Esfera de apoio (ball transfer): corpo livre de atrito, rola em qualquer direcao -->
+    <xacro:macro name="caster_ball" params="name y">
         <link name="${name}">
             <visual>
-                <origin xyz="0 0 0" rpy="${rpy}"/>
                 <geometry><mesh filename="${meshes}/12mmball__revolve1.stl"/></geometry>
                 <material name="grey"/>
@@ -65,6 +99,8 @@
             </collision>
             <inertial>
-                <mass value="0.005"/>
-                <inertia ixx="1e-7" ixy="0" ixz="0" iyy="1e-7" iyz="0" izz="1e-7"/>
+                <mass value="${caster_ball_mass}"/>
+                <inertia ixx="${0.4*caster_ball_mass*caster_ball_radius*caster_ball_radius}" ixy="0" ixz="0"
+                         iyy="${0.4*caster_ball_mass*caster_ball_radius*caster_ball_radius}" iyz="0"
+                         izz="${0.4*caster_ball_mass*caster_ball_radius*caster_ball_radius}"/>
             </inertial>
         </link>
@@ -72,55 +108,76 @@
             <parent link="chassis"/>
             <child link="${name}"/>
-            <origin xyz="${xyz}" rpy="0 0 0"/>
+            <origin xyz="0 ${y} ${caster_z}" rpy="0 0 0"/>
         </joint>
     </xacro:macro>
     <!-- ================= LINKS ================= -->
     <link name="base_link"/>
-    <!-- chassis: tudo o que e fixo no CAD (frame do Onshape) -->
+    <!-- chassis: tudo o que e rigido no CAD. Poses no plate frame (mm convertidos para m). -->
     <link name="chassis">
-        <xacro:chassis_visual mesh="base.stl" xyz="-0.00104301 -0.00775804 -0.00550781" rpy="0.000156777 0.0169755 0.042698"/>
-        <xacro:chassis_visual mesh="resto.stl" xyz="-0.000703692 -0.00774668 0.0144893" rpy="0.000156777 0.0169755 0.042698"/>
-        <xacro:chassis_visual mesh="n20_mini_micro_metall_gear_motor.stl" xyz="0.0294437 -0.00645663 0.000975149" rpy="0.000156777 0.0169755 0.042698" material="grey"/>
-        <xacro:chassis_visual mesh="n20_mini_micro_metall_gear_motor.stl" xyz="-0.0312922 -0.00905151 0.00200721" rpy="-0.000156777 -0.0169755 -3.09889" material="grey"/>
-        <xacro:chassis_visual mesh="eletroiman.stl" xyz="0.000994645 -0.0538637 -0.00151562" rpy="1.57095 0.0169755 0.042698" material="orange"/>
-        <xacro:chassis_visual mesh="rp_lidar.stl" xyz="0.123908 -0.080762 -0.657373" rpy="1.55382 0.000156754 -1.5281" material="grey"/>
-        <xacro:chassis_visual mesh="casterballwheelbody__cut_extrude6.stl" xyz="0.00028842 -0.0458832 -0.0230113" rpy="0.000156777 0.0169755 0.042698" material="white"/>
-        <xacro:chassis_visual mesh="casterballwheellid__cut_extrude2.stl" xyz="0.000469237 -0.0458607 -0.0123128" rpy="-0.0164377 -0.00424196 -1.78986" material="white"/>
-        <xacro:chassis_visual mesh="casterballwheelbody__cut_extrude6.stl" xyz="-0.00288046 0.0283327 -0.0228996" rpy="0.000156777 0.0169755 0.042698" material="white"/>
-        <xacro:chassis_visual mesh="casterballwheellid__cut_extrude2.stl" xyz="-0.00269965 0.0283552 -0.0122012" rpy="-0.0164377 -0.00424196 -1.78986" material="white"/>
-        <!-- colisao simplificada: so a placa da base -->
-        <collision>
-            <origin xyz="-0.00104301 -0.00775804 -0.00550781" rpy="0.000156777 0.0169755 0.042698"/>
-            <geometry><mesh filename="${meshes}/base.stl"/></geometry>
+        <xacro:chassis_visual mesh="base.stl"  xyz="0 0 0" rpy="0 0 0"/>
+        <xacro:chassis_visual mesh="resto.stl" xyz="0 0 0.02" rpy="0 0 0"/>
+        <xacro:chassis_visual mesh="n20_mini_micro_metall_gear_motor.stl" xyz="0.0304 0 0.007" rpy="0 0 0" material="grey"/>
+        <xacro:chassis_visual mesh="n20_mini_micro_metall_gear_motor.stl" xyz="-0.0304 0 0.007" rpy="0 0 ${-pi}" material="grey"/>
+        <xacro:chassis_visual mesh="eletroiman.stl" xyz="0 -0.04615 0.004" rpy="${pi/2} 0 0" material="orange"/>
+        <!-- a mesh do LIDAR tem a origem longe do corpo; esta pose poe-no assente no topo do 'resto' -->
+        <xacro:chassis_visual mesh="rp_lidar.stl" xyz="0.13277 -0.07837 -0.64969" rpy="${pi/2} 0 ${-pi/2}" material="grey"/>
+        <xacro:chassis_visual mesh="casterballwheelbody__cut_extrude6.stl" xyz="0 ${caster_front_y} -0.0175" rpy="0 0 0" material="white"/>
+        <xacro:chassis_visual mesh="casterballwheellid__cut_extrude2.stl"  xyz="0 ${caster_front_y} -0.0068" rpy="0 0 -1.83259" material="white"/>
+        <xacro:chassis_visual mesh="casterballwheelbody__cut_extrude6.stl" xyz="0 ${caster_rear_y} -0.0174" rpy="0 0 0" material="white"/>
+        <xacro:chassis_visual mesh="casterballwheellid__cut_extrude2.stl"  xyz="0 ${caster_rear_y} -0.0067" rpy="0 0 -1.83259" material="white"/>
+        <!-- COLISOES simplificadas (primitivas): placa + corpo + caixa do LIDAR + cabeca do LIDAR + iman.
+             Antes so existia a placa, por isso o robo atravessava paredes a altura do corpo/LIDAR. -->
+        <collision name="plate_col">
+            <origin xyz="0 0 0.0065" rpy="0 0 0"/>
+            <geometry><box size="0.080 0.0963 0.027"/></geometry>
         </collision>
-        <!-- TODO: massa e inercia reais (atribuir materiais no Onshape ou medir) -->
+        <collision name="body_col">
+            <origin xyz="0 0 0.045" rpy="0 0 0"/>
+            <geometry><box size="0.080 0.0963 0.050"/></geometry>
+        </collision>
+        <collision name="lidar_housing_col">
+            <origin xyz="-0.0001 -0.0025 0.08345" rpy="0 0 0"/>
+            <geometry><box size="0.0703 0.0961 0.0229"/></geometry>
+        </collision>
+        <collision name="lidar_head_col">
+            <origin xyz="0 0.0124 0.1092" rpy="0 0 0"/>
+            <geometry><cylinder radius="0.0347" length="0.0286"/></geometry>
+        </collision>
+        <collision name="magnet_col">
+            <origin xyz="0 -0.05365 0.004" rpy="${pi/2} 0 0"/>
+            <geometry><cylinder radius="0.01" length="0.015"/></geometry>
+        </collision>
+        <!-- massa/CM/inercia calculados a partir das meshes: ver tools/mass_budget.py -->
         <inertial>
-            <origin xyz="0 -0.01 0" rpy="0 0 0"/>
+            <origin xyz="${chassis_com}" rpy="0 0 0"/>
             <mass value="${chassis_mass}"/>
-            <inertia ixx="${chassis_mass/12*(0.1*0.1+0.03*0.03)}" ixy="0" ixz="0"
-                     iyy="${chassis_mass/12*(0.1*0.1+0.03*0.03)}" iyz="0"
-                     izz="${chassis_mass/12*(0.1*0.1+0.1*0.1)}"/>
+            <inertia ixx="${chassis_ixx}" ixy="${chassis_ixy}" ixz="${chassis_ixz}"
+                     iyy="${chassis_iyy}" iyz="${chassis_iyz}" izz="${chassis_izz}"/>
         </inertial>
     </link>
+    <!-- plate frame: 7 mm abaixo do eixo, rodado 90 graus (frente do CAD = -Y  ->  +X do ROS) -->
     <joint name="chassis_joint" type="fixed">
         <parent link="base_link"/>
         <child link="chassis"/>
-        <origin xyz="0 0 0" rpy="0 0 ${chassis_yaw}"/>
+        <origin xyz="0 0 ${-axle_height_in_plate}" rpy="0 0 ${pi/2}"/>
     </joint>
-    <!-- ================= RODAS (continuous) ================= -->
-    <!-- Esquerda = roda_2 do CAD (x>0), direita = roda do CAD (x<0).
-         Eixo da esquerda invertido para que velocidade positiva = andar para a frente. -->
-    <xacro:wheel name="left"  xyz="0.0404288 -0.00591039 0.000788417" rpy="0.0213475 -1.55382 0.0213475" axis="0 0 -1"/>
-    <xacro:wheel name="right" xyz="-0.0422773 -0.00959774 0.00219389" rpy="-3.12025 -1.55382 0.0213475" axis="0 0 1"/>
+    <!-- ================= RODAS (continuous) =================
+         Esquerda = +Y, direita = -Y. Os dois eixos apontam para +Y (Z do link),
+         logo velocidade positiva nas duas = frente.
+         vis_z/vis_roll: a mesh roda.stl vai de z=0 (face interior) a z=+8 mm (face exterior);
+         na direita o exterior e -Z do link, por isso a mesh e virada 180 graus. -->
+    <xacro:wheel name="left"  y="${wheel_y}"  vis_z="${-wheel_width/2}" vis_roll="0"/>
+    <xacro:wheel name="right" y="${-wheel_y}" vis_z="${wheel_width/2}"  vis_roll="${pi}"/>
     <!-- ================= ESFERAS (casters) ================= -->
-    <xacro:caster_ball name="caster_a" xyz="0.000330117 -0.0458654 -0.0205116" rpy="-0.00424253 0.0164375 -0.219138"/>
-    <xacro:caster_ball name="caster_b" xyz="-0.00283877 0.0283506 -0.0204" rpy="-0.00424253 0.0164375 -0.219138"/>
+    <xacro:caster_ball name="caster_front" y="${caster_front_y}"/>
+    <xacro:caster_ball name="caster_rear"  y="${caster_rear_y}"/>
     <!-- ================= LIDAR ================= -->
-    <!-- visual do LIDAR no chassis (pose do export; a mesh tem a origem longe do corpo) -->
+    <!-- laser_frame ligado ao base_link (NAO ao chassis): o eixo X do laser tem de apontar
+         para a frente do robo, senao o angulo 0 do scan fica virado 90 graus para o lado. -->
     <link name="laser_frame"/>
     <joint name="laser_joint" type="fixed">
-        <parent link="chassis"/>
+        <parent link="base_link"/>
         <child link="laser_frame"/>
-        <origin xyz="${lidar_xyz}" rpy="0 0 0"/>
+        <origin xyz="${lidar_x} ${lidar_y} ${lidar_z}" rpy="0 0 0"/>
     </joint>
 </robot>
